Commit message: wip

File: examples/pendulum_kinematic/pendulum.urdf (robot description, URDF)
Before this commit: robot pendulum, 3 links, 2 joints
Joints:
- joint roottoseg1: axis 1. 0. 0. -> 1 0 0
- joint seg1toseg2: axis 1. 0. 0. -> 1 0 0; origin xyz=0. 0. -1. -> xyz=0 0 -1

Commit message: updating gif

File: examples/pendulum_kinematic/pendulum.urdf (robot description, URDF)
Before this commit: robot pendulum, 3 links, 2 joints
Links:
- link segment1: geometry visual box size=0.2 0.2 1
Joints:
- joint seg1toseg2: origin xyz=0 0 -1 -> xyz=1 0 0

Commit message: some examples and wiki update. pending permission to use jumping model

File: examples/pendulum_kinematic/pendulum.urdf (robot description, URDF)
Before this commit: robot pendulum, 3 links, 2 joints
Joints:
- joint seg1toseg2: origin xyz=1 0 0 -> xyz=0 0 1
